Commit message: Add lidar and no map move base option

File: catkin_ws/src/ottobot_description/urdf/kinect.urdf.xacro (robot description, xacro)
@@ -3,5 +3,5 @@
 <!-- https://github.com/${parent}turtlebot/${parent}turtlebot/blob/hydro/${parent}turtlebot_description/urdf/sensors/kinect.urdf.xacro -->
 <robot name="sensor_kinect" xmlns:xacro="http://www.ros.org/wiki/xacro">
-    <xacro:include filename="$(find ottobot_description)/urdf/kinect.gazebo.urdf.xacro"/>
+    <xacro:include filename="$(find ottobot_description)/urdf/kinect.gazebo.xacro"/>
     <xacro:macro name="sensor_kinect" params="parent">
         <joint name="camera_rgb_joint" type="fixed">
@@ -81,5 +81,5 @@
         </link>
         <!-- Kinect sensor for simulation defined in kinect.gazebo.urdf.xacro -->
-        <xacro:ottobot_sim_3dsensor />
+        <xacro:sim_gazebo_kinect />
     </xacro:macro>
 </robot>

File: catkin_ws/src/ottobot_description/urdf/ottobot.urdf.xacro (robot description, xacro)
@@ -4,7 +4,12 @@
     <!-- SUB-COMPONENTS -->
     <xacro:include filename="$(find ottobot_description)/urdf/ottobot_wheel.urdf.xacro" />
-    <xacro:arg name="use_kinect" default="false" />
-    <xacro:include filename="$(find ottobot_description)/urdf/kinect.urdf.xacro" />
-    <xacro:arg name="use_lidar" default="false" />
+    <xacro:arg name="enable_kinect" default="false" />
+    <xacro:if value="$(arg enable_kinect)">
+        <xacro:include filename="$(find ottobot_description)/urdf/kinect.urdf.xacro" />
+    </xacro:if>
+    <xacro:arg name="enable_lidar" default="false" />
+    <xacro:if value="$(arg enable_lidar)">
+        <xacro:include filename="$(find ottobot_description)/urdf/a1rplidar.urdf.xacro" />
+    </xacro:if>
     <!-- PROPERTIES -->
     <xacro:property name="M_PI" value="3.14159"/>
@@ -28,4 +33,11 @@
 	<xacro:property name="cam_op" value="0" />
 	<xacro:property name="cam_oy" value="0" />
+    <!-- A1 Lidar pose -->
+    <xacro:property name="lidar_px" value="0.06" />
+	<xacro:property name="lidar_py" value="0" />
+	<xacro:property name="lidar_pz" value="${0.04 + chassis_height/2}" />
+	<xacro:property name="lidar_or" value="0" />
+	<xacro:property name="lidar_op" value="0" />
+	<xacro:property name="lidar_oy" value="0" />
     <!-- PLUGINS -->
     <xacro:include filename="$(find ottobot_description)/urdf/ottobot.gazebo.xacro" />
@@ -83,6 +95,9 @@
         <origin xyz="-0.031 0.035 0.183" rpy="0 0 0"/>
     </joint>
-    <xacro:if value="$(arg use_kinect)">
+    <xacro:if value="$(arg enable_kinect)">
         <xacro:sensor_kinect parent="chassis"></xacro:sensor_kinect>
+    </xacro:if>
+    <xacro:if value="$(arg enable_lidar)">
+        <xacro:sensor_lidar parent="chassis"></xacro:sensor_lidar>
     </xacro:if>
     <!-- COLORS - - - - - - - - -->
