Commit message: fixed frame names

File: catkin_ws/src/ottobot_description/urdf/a1rplidar.gazebo.xacro (robot description, xacro)
@@ -3,5 +3,5 @@
   <!-- RPLIDAR A1 Lidar -->
   <xacro:macro name="sim_gazebo_a1rplidar">
-    <gazebo reference="lidar_link">
+    <gazebo reference="lidar">
     <!-- http://sdformat.org/spec?ver=1.7&elem=sensor#sensor_lidar -->
         <sensor type="ray" name="head_a1rplidar_sensor">
@@ -35,5 +35,5 @@
             <plugin name="gazebo_ros_head_a1rplidar_controller" filename="libgazebo_ros_laser.so">
                 <topicName>scan</topicName>
-                <frameName>lidar_link</frameName>
+                <frameName>lidar</frameName>
             </plugin>
         </sensor>

File: catkin_ws/src/ottobot_description/urdf/a1rplidar.urdf.xacro (robot description, xacro)
@@ -6,7 +6,7 @@
             <origin xyz="${lidar_px} ${lidar_py} ${lidar_pz}" rpy="${lidar_or} ${lidar_op} ${lidar_oy}"/>
             <parent link="${parent}"/>
-            <child link="lidar_link" />
+            <child link="lidar" />
         </joint>
-        <link name="lidar_link">
+        <link name="lidar">
             <collision>
                 <geometry>

File: catkin_ws/src/ottobot_description/urdf/ottobot.gazebo.xacro (robot description, xacro)
@@ -7,25 +7,3 @@
         </plugin>
     </gazebo>
-    <!-- IMU -->
-    <!-- http://gazebosim.org/tutorials?tut=ros_gzplugins#IMUsensor(GazeboRosImuSensor) -->
-    <!-- https://cdn-shop.adafruit.com/datasheets/BST_BNO055_DS000_12.pdf -->
-    <gazebo reference="imu_link">
-        <gravity>true</gravity>
-        <sensor name="imu_sensor" type="imu">
-            <always_on>true</always_on>
-            <update_rate>100</update_rate>
-            <visualize>true</visualize>
-            <topic>__default_topic__</topic>
-            <plugin filename="libgazebo_ros_imu_sensor.so" name="imu_plugin">
-                <topicName>imu</topicName>
-                <bodyName>imu_link</bodyName>
-                <updateRateHZ>10.0</updateRateHZ>
-                <gaussianNoise>0.0</gaussianNoise>
-                <xyzOffset>0 0 0</xyzOffset>
-                <rpyOffset>0 0 0</rpyOffset>
-                <frameName>imu_link</frameName>
-                <initialOrientationAsReference>false</initialOrientationAsReference>
-            </plugin>
-        </sensor>
-    </gazebo>
 </robot>

File: catkin_ws/src/ottobot_description/urdf/ottobot.urdf.xacro (robot description, xacro)
@@ -4,4 +4,5 @@
     <!-- SUB-COMPONENTS -->
     <xacro:include filename="$(find ottobot_description)/urdf/ottobot_wheel.urdf.xacro" />
+    <xacro:include filename="$(find ottobot_description)/urdf/bno055imu.urdf.xacro" />
     <xacro:arg name="enable_kinect" default="false" />
     <xacro:if value="$(arg enable_kinect)">
@@ -89,10 +90,5 @@
     </xacro:ottobot_wheel>
     <!-- SENSORS - - - - - - - - -->
-    <link name="imu_link"/>
-    <joint name="imu_joint" type="fixed">
-        <parent link="${parent}"/>
-        <child link="imu_link"/>
-        <origin xyz="-0.031 0.035 0.183" rpy="0 0 0"/>
-    </joint>
+    <xacro:sensor_imu parent="chassis"></xacro:sensor_imu>
     <xacro:if value="$(arg enable_kinect)">
         <xacro:sensor_kinect parent="chassis"></xacro:sensor_kinect>
