Commit message: Fixed urdf for lidar

File: catkin_ws/src/ottobot_description/urdf/a1rplidar.urdf.xacro (robot description, xacro)
@@ -2,22 +2,27 @@
 <robot name="sensor_lidar" xmlns:xacro="http://www.ros.org/wiki/xacro">
     <xacro:include filename="$(find ottobot_description)/urdf/a1rplidar.gazebo.xacro"/>
+    <xacro:property name="frame_height" value="0.032" />
+    <xacro:property name="head_height" value="0.024" />
     <xacro:macro name="sensor_lidar" params="parent">
-        <joint name="lidar_joint" type="fixed">
+        <joint name="lidar_base_joint" type="fixed">
             <origin xyz="${lidar_px} ${lidar_py} ${lidar_pz}" rpy="${lidar_or} ${lidar_op} ${lidar_oy}"/>
             <parent link="${parent}"/>
-            <child link="lidar" />
+            <child link="lidar_base" />
         </joint>
-        <link name="lidar">
+        <link name="lidar_base">
             <collision>
+                <origin xyz="0 0 ${frame_height / 2}" rpy="0 0 0"/>
                 <geometry>
-                    <box size="0.0985 0.07 0.06" />
+                    <box size="0.0985 0.07 ${frame_height}" />
                 </geometry>
             </collision>
             <visual>
+                <origin xyz="0 0 ${frame_height / 2}" rpy="0 0 0"/>
                 <geometry>
-                    <box size="0.0985 0.07 0.06" />
+                    <box size="0.0985 0.07 ${frame_height}" />
                 </geometry>
             </visual>
             <inertial>
+                <origin xyz="0 0 ${(frame_height + head_height) / 2}"/>
                 <mass value="0.17" />
                 <origin xyz="0 0 0" rpy="0 0 0"/>
@@ -25,4 +30,23 @@
             </inertial>
         </link>
+        <joint name="lidar_head_joint" type="fixed">
+            <origin xyz="-0.013350 0 ${frame_height}" rpy="0 0 0" />
+            <parent link="lidar_base" />
+            <child link="lidar" />
+        </joint>
+        <link name="lidar">
+            <origin xyz="0 0 ${head_height / 2}" rpy="0 0 0"/>
+            <collision>
+                <geometry>
+                    <cylinder radius="0.035" length="${head_height}"/>
+                </geometry>
+            </collision>
+            <visual>
+                <origin xyz="0 0 ${head_height / 2}" rpy="0 0 0"/>
+                <geometry>
+                    <cylinder radius="0.035" length="${head_height}"/>
+                </geometry>
+            </visual>
+        </link>
         <!-- Lidar sensor for simulation defined in a1rplidar.gazebo.xacro -->
         <xacro:sim_gazebo_a1rplidar />

File: catkin_ws/src/ottobot_description/urdf/ottobot.urdf.xacro (robot description, xacro)
@@ -39,5 +39,5 @@
     <xacro:property name="lidar_px" value="0.06" />
 	<xacro:property name="lidar_py" value="0" />
-	<xacro:property name="lidar_pz" value="${0.04 + chassis_height/2}" />
+	<xacro:property name="lidar_pz" value="${0.012 + chassis_height/2}" />
 	<xacro:property name="lidar_or" value="0" />
 	<xacro:property name="lidar_op" value="0" />
