Commit message: IMU position fixed

File: catkin_ws/src/ottobot_description/urdf/bno055imu.urdf.xacro (robot description, xacro)
@@ -3,10 +3,17 @@
     <xacro:include filename="$(find ottobot_description)/urdf/bno055imu.gazebo.xacro"/>
     <xacro:macro name="sensor_imu" params="parent">
-        <link name="imu"/>
         <joint name="imu_joint" type="fixed">
+            <origin xyz="${imu_px} ${imu_py} ${imu_pz}" rpy="${imu_or} ${imu_op} ${imu_oy}"/>
             <parent link="${parent}"/>
             <child link="imu"/>
-            <origin xyz="-0.031 0.035 0.183" rpy="0 0 0"/>
         </joint>
+        <link name="imu">
+            <visual>
+                <origin xyz="0 0 0" rpy="0 0 0"/>
+                <geometry>
+                    <box size="0.027 0.02 0.0025" />
+                </geometry>
+            </visual>
+        </link>
         <!-- IMU sensor for simulation defined in bno055imu.gazebo.xacro -->
         <xacro:sim_gazebo_bno055imu />

File: catkin_ws/src/ottobot_description/urdf/ottobot.urdf.xacro (robot description, xacro)
@@ -29,4 +29,11 @@
     <xacro:property name="wheel_left_offset" value="0.125" />
     <xacro:property name="wheel_vert_offset" value="${-chassis_gnd_clearance - chassis_height/2 + wheel_rad}" />
+    <!-- IMU pose -->
+    <xacro:property name="imu_px" value="-0.032" />
+	<xacro:property name="imu_py" value="-0.035" />
+	<xacro:property name="imu_pz" value="${0.039 + chassis_height/2}" />
+	<xacro:property name="imu_or" value="0" />
+	<xacro:property name="imu_op" value="0" />
+	<xacro:property name="imu_oy" value="${M_PI}" />
     <!-- Kinect pose -->
     <xacro:property name="cam_px" value="${chassis_length / 2}" />
