Commit message: Updated to match Wild Thumper

File: catkin_ws/src/ottobot_description/urdf/ottobot.urdf.xacro (robot description, xacro)
@@ -8,17 +8,19 @@
     <xacro:property name="M_PI" value="3.14159"/>
     <xacro:property name="parent" value="robot_footprint" />
-    <xacro:property name="chassis_mass" value="15.0" />
-    <xacro:property name="chassis_height" value="0.12" />
-    <xacro:property name="chassis_length" value="0.4" />
-    <xacro:property name="chassis_width" value="0.2" />
-    <xacro:property name="wheel_mass" value="1.5" />
-    <xacro:property name="wheel_width" value="0.06" />
-    <xacro:property name="wheel_rad" value="0.1" />
-    <xacro:property name="wheel_forward_offset" value="0.13" />
-    <xacro:property name="wheel_left_offset" value="${chassis_width/2 + 0.05}" />
+    <xacro:property name="chassis_mass" value="2.0" />
+    <xacro:property name="chassis_height" value="0.095" />
+    <xacro:property name="chassis_length" value="0.23" />
+    <xacro:property name="chassis_width" value="0.12" />
+    <xacro:property name="chassis_gnd_clearance" value="0.05" />
+    <xacro:property name="wheel_mass" value="0.186" />
+    <xacro:property name="wheel_width" value="0.062" />
+    <xacro:property name="wheel_rad" value="0.063" />
+    <xacro:property name="wheel_forward_offset" value="0.075" />
+    <xacro:property name="wheel_left_offset" value="0.125" />
+    <xacro:property name="wheel_vert_offset" value="${-chassis_gnd_clearance - chassis_height/2 + wheel_rad}" />
     <!-- Kinect pose -->
-    <xacro:property name="cam_px" value="-0.087" />
-	<xacro:property name="cam_py" value="-0.0125" /> Y varies for different configurations. get sets in sensors_urdf
-	<xacro:property name="cam_pz" value="0.2870" />
+    <xacro:property name="cam_px" value="${chassis_length / 2}" />
+	<xacro:property name="cam_py" value="0" />
+	<xacro:property name="cam_pz" value="${0.05 + chassis_height/2}" />
 	<xacro:property name="cam_or" value="0" />
 	<xacro:property name="cam_op" value="0" />
@@ -29,5 +31,5 @@
     <link name="${parent}"></link>
     <joint name="${parent}_joint" type="fixed">
-        <origin xyz="0 0 ${wheel_rad}" rpy="0 0 0" />
+        <origin xyz="0 0 ${chassis_gnd_clearance + chassis_height/2}" rpy="0 0 0" />
         <parent link="${parent}"/>
         <child link="chassis" />
@@ -61,17 +63,17 @@
     <!-- Format from https://github.com/husky/husky/blob/melodic-devel/husky_description/urdf/husky.urdf.xacro -->
     <xacro:ottobot_wheel wheel_prefix="front_left">
-        <origin xyz="${wheel_forward_offset} ${wheel_left_offset} 0" rpy="0 0 0" />
+        <origin xyz="${wheel_forward_offset} ${wheel_left_offset} ${wheel_vert_offset}" rpy="0 0 0" />
     </xacro:ottobot_wheel>
     <xacro:ottobot_wheel wheel_prefix="front_right">
-        <origin xyz="${wheel_forward_offset} -${wheel_left_offset} 0" rpy="0 0 0" />
+        <origin xyz="${wheel_forward_offset} -${wheel_left_offset} ${wheel_vert_offset}" rpy="0 0 0" />
     </xacro:ottobot_wheel>
     <xacro:ottobot_wheel wheel_prefix="back_left">
-        <origin xyz="-${wheel_forward_offset} ${wheel_left_offset} 0" rpy="0 0 0" />
+        <origin xyz="-${wheel_forward_offset} ${wheel_left_offset} ${wheel_vert_offset}" rpy="0 0 0" />
     </xacro:ottobot_wheel>
     <xacro:ottobot_wheel wheel_prefix="back_right">
-        <origin xyz="-${wheel_forward_offset} -${wheel_left_offset} 0" rpy="0 0 0" />
+        <origin xyz="-${wheel_forward_offset} -${wheel_left_offset} ${wheel_vert_offset}" rpy="0 0 0" />
     </xacro:ottobot_wheel>
     <!-- SENSORS - - - - - - - - -->
-    <xacro:sensor_kinect parent="${parent}">
+    <xacro:sensor_kinect parent="chassis">
     </xacro:sensor_kinect>
     <!-- COLORS - - - - - - - - -->

File: catkin_ws/src/ottobot_description/urdf/ottobot_wheel.urdf.xacro (robot description, xacro)
@@ -35,5 +35,5 @@
 				</xacro:unless>
                 <geometry>
-                    <sphere radius="0.02"/>
+                    <sphere radius="0.005"/>
                 </geometry>
             </visual>

Commit message: Testing setup

File: catkin_ws/src/ottobot_description/urdf/ottobot.urdf.xacro (robot description, xacro)
@@ -4,5 +4,7 @@
     <!-- SUB-COMPONENTS -->
     <xacro:include filename="$(find ottobot_description)/urdf/ottobot_wheel.urdf.xacro" />
+    <xacro:arg name="use_kinect" default="false" />
     <xacro:include filename="$(find ottobot_description)/urdf/kinect.urdf.xacro" />
+    <xacro:arg name="use_lidar" default="false" />
     <!-- PROPERTIES -->
     <xacro:property name="M_PI" value="3.14159"/>
@@ -27,5 +29,5 @@
 	<xacro:property name="cam_oy" value="0" />
     <!-- PLUGINS -->
-    <xacro:include filename="$(find ottobot_description)/urdf/roscontrol.gazebo.xacro" />
+    <xacro:include filename="$(find ottobot_description)/urdf/ottobot.gazebo.xacro" />
     <!-- PARTS -->
     <link name="${parent}"></link>
@@ -75,6 +77,13 @@
     </xacro:ottobot_wheel>
     <!-- SENSORS - - - - - - - - -->
-    <xacro:sensor_kinect parent="chassis">
-    </xacro:sensor_kinect>
+    <link name="imu_link"/>
+    <joint name="imu_joint" type="fixed">
+        <parent link="${parent}"/>
+        <child link="imu_link"/>
+        <origin xyz="-0.031 0.035 0.183" rpy="0 0 0"/>
+    </joint>
+    <xacro:if value="$(arg use_kinect)">
+        <xacro:sensor_kinect parent="chassis"></xacro:sensor_kinect>
+    </xacro:if>
     <!-- COLORS - - - - - - - - -->
     <gazebo reference="left_wheel">

Commit message: Rotate lidar by 180deg

File: catkin_ws/src/ottobot_description/urdf/ottobot.urdf.xacro (robot description, xacro)
@@ -14,5 +14,7 @@
     </xacro:if>
     <!-- PROPERTIES -->
-    <xacro:property name="M_PI" value="3.14159"/>
+    <xacro:property name="M_PI"   value="3.141592653"/>
+    <xacro:property name="M_2_PI" value="6.283185307"/>
+    <xacro:property name="M_PI_2" value="1.570796326"/>
     <xacro:property name="parent" value="robot_footprint" />
     <xacro:property name="chassis_mass" value="2.0" />
@@ -40,5 +42,5 @@
 	<xacro:property name="lidar_or" value="0" />
 	<xacro:property name="lidar_op" value="0" />
-	<xacro:property name="lidar_oy" value="0" />
+	<xacro:property name="lidar_oy" value="${M_PI_2}" />
     <!-- PLUGINS -->
     <xacro:include filename="$(find ottobot_description)/urdf/ottobot.gazebo.xacro" />

Commit message: Fix rotation

File: catkin_ws/src/ottobot_description/urdf/ottobot.urdf.xacro (robot description, xacro)
@@ -42,5 +42,5 @@
 	<xacro:property name="lidar_or" value="0" />
 	<xacro:property name="lidar_op" value="0" />
-	<xacro:property name="lidar_oy" value="${M_PI_2}" />
+	<xacro:property name="lidar_oy" value="${M_PI}" />
     <!-- PLUGINS -->
     <xacro:include filename="$(find ottobot_description)/urdf/ottobot.gazebo.xacro" />

Commit message: debug

File: catkin_ws/src/ottobot_description/urdf/ottobot.urdf.xacro (robot description, xacro)
@@ -42,5 +42,5 @@
 	<xacro:property name="lidar_or" value="0" />
 	<xacro:property name="lidar_op" value="0" />
-	<xacro:property name="lidar_oy" value="${M_PI}" />
+	<xacro:property name="lidar_oy" value="0" />
     <!-- PLUGINS -->
     <xacro:include filename="$(find ottobot_description)/urdf/ottobot.gazebo.xacro" />

Commit message: angle

File: catkin_ws/src/ottobot_description/urdf/ottobot.urdf.xacro (robot description, xacro)
@@ -42,5 +42,5 @@
 	<xacro:property name="lidar_or" value="0" />
 	<xacro:property name="lidar_op" value="0" />
-	<xacro:property name="lidar_oy" value="0" />
+	<xacro:property name="lidar_oy" value="${M_PI}" />
     <!-- PLUGINS -->
     <xacro:include filename="$(find ottobot_description)/urdf/ottobot.gazebo.xacro" />

Commit message: Tuning controller params

File: catkin_ws/src/ottobot_description/urdf/ottobot.urdf.xacro (robot description, xacro)
@@ -25,5 +25,5 @@
     <xacro:property name="wheel_mass" value="0.186" />
     <xacro:property name="wheel_width" value="0.062" />
-    <xacro:property name="wheel_rad" value="0.063" />
+    <xacro:property name="wheel_rad" value="0.064" />
     <xacro:property name="wheel_forward_offset" value="0.075" />
     <xacro:property name="wheel_left_offset" value="0.125" />

File: catkin_ws/src/ottobot_description/urdf/ottobot_wheel.urdf.xacro (robot description, xacro)
@@ -42,6 +42,6 @@
 			<mu1 value="0.9"/>
 			<mu2 value="0.9"/>
-			<kp value="1000000.0" />
-			<kd value="10.0" />
+			<kp value="1.5" />
+			<ki value="15.0" />
 			<!-- <fdir1 value="0 0 1"/> -->
 		</gazebo>
